Commit message: Added custom world

File: src/vision_line_follower/urdf/my_robot.urdf.xacro (robot description, xacro)
@@ -32,5 +32,104 @@
     </inertial>
   </link>
-  <!-- Camera Link -->
+    <!-- Left wheel -->
+    <link name="left_wheel">
+      <visual>
+        <origin xyz="0 0 0" rpy="1.5708 0 0"/>
+        <geometry>
+          <cylinder length="${wheel_width}" radius="${wheel_radius}"/>
+        </geometry>
+        <material name="black">
+          <color rgba="0 0 0 1"/>
+        </material>
+      </visual>
+      <collision>
+        <origin xyz="0 0 0" rpy="1.5708 0 0"/>
+        <geometry>
+          <cylinder length="${wheel_width}" radius="${wheel_radius}"/>
+        </geometry>
+      </collision>
+      <inertial>
+        <origin xyz="0 0 0" rpy="0 0 0"/>
+        <mass value="0.1"/>
+        <inertia ixx="0.0001" ixy="0.0" ixz="0.0"
+                 iyy="0.0001" iyz="0.0"
+                 izz="0.0001"/>
+      </inertial>
+    </link>
+    <gazebo reference="left_wheel">
+      <material>Gazebo/Black</material>
+    </gazebo>
+    <!-- Right wheel -->
+    <link name="right_wheel">
+      <visual>
+        <origin xyz="0 0 0" rpy="1.5708 0 0"/>
+        <geometry>
+          <cylinder length="${wheel_width}" radius="${wheel_radius}"/>
+        </geometry>
+        <material name="black">
+          <color rgba="0 0 0 1"/>
+        </material>
+      </visual>
+      <collision>
+        <origin xyz="0 0 0" rpy="1.5708 0 0"/>
+        <geometry>
+          <cylinder length="${wheel_width}" radius="${wheel_radius}"/>
+        </geometry>
+      </collision>
+      <inertial>
+        <origin xyz="0 0 0" rpy="0 0 0"/>
+        <mass value="0.1"/>
+        <inertia ixx="0.0001" ixy="0.0" ixz="0.0"
+                 iyy="0.0001" iyz="0.0"
+                 izz="0.0001"/>
+      </inertial>
+    </link>
+    <gazebo reference="right_wheel">
+      <material>Gazebo/Black</material>
+    </gazebo>
+  <!-- Joints for wheels -->
+  <joint name="left_wheel_joint" type="continuous">
+    <parent link="base_link"/>
+    <child link="left_wheel"/>
+    <origin xyz="-${body_length/3} ${body_width/2 + wheel_width/2} ${wheel_radius/2}" rpy="0 0 0"/>
+    <axis xyz="0 1 0"/>
+  </joint>
+  <joint name="right_wheel_joint" type="continuous">
+    <parent link="base_link"/>
+    <child link="right_wheel"/>
+    <origin xyz="-${body_length/3} -${body_width/2 + wheel_width/2} ${wheel_radius/2}" rpy="0 0 0"/>
+    <axis xyz="0 1 0"/>
+  </joint>
+  <!-- Front Caster Wheel -->
+  <link name="caster_wheel">
+    <visual>
+      <geometry>
+        <sphere radius="0.03"/>
+      </geometry>
+      <origin xyz="0 0 0" rpy="0 0 0"/>
+      <material name="grey">
+        <color rgba="0.5 0.5 0.5 1"/>
+      </material>
+    </visual>
+    <collision>
+      <geometry>
+        <sphere radius="0.03"/>
+      </geometry>
+      <origin xyz="0 0 0" rpy="0 0 0"/>
+    </collision>
+    <inertial>
+      <mass value="0.1"/>
+      <inertia ixx="0.00005" ixy="0.0" ixz="0.0"
+               iyy="0.00005" iyz="0.0"
+               izz="0.00005"/>
+      <origin xyz="0 0 0" rpy="0 0 0"/>
+    </inertial>
+  </link>
+  <joint name="caster_joint" type="fixed">
+    <parent link="base_link"/>
+    <child link="caster_wheel"/>
+    <origin xyz="0.05 0 0" rpy="0 0 0"/>
+  </joint>
+  <!-- Camera link -->
   <link name="camera_link">
     <visual>
@@ -44,5 +143,4 @@
     </visual>
   </link>
-  <!-- Joint: base_link to camera_link -->
   <joint name="camera_joint" type="fixed">
     <parent link="base_link"/>
@@ -50,5 +148,5 @@
     <origin xyz="0.1 0 ${body_height + 0.025}" rpy="0 0 0"/>
   </joint>
-  <!-- Gazebo camera plugin -->
+  <!-- Gazebo plugin for camera -->
   <gazebo reference="camera_link">
     <sensor type="camera" name="camera_sensor">

Commit message: Added functionality to follow line and scan qr codes to take decisions

File: src/vision_line_follower/urdf/my_robot.urdf.xacro (robot description, xacro)
@@ -10,5 +10,5 @@
   <link name="base_link">
     <visual>
-      <origin xyz="0 0 ${body_height / 2}" rpy="0 0 0"/>
+      <origin xyz="0 0 ${wheel_radius + body_height / 2}" rpy="0 0 0"/>
       <geometry>
         <box size="${body_length} ${body_width} ${body_height}"/>
@@ -89,18 +89,20 @@
     </gazebo>
   <!-- Joints for wheels -->
+  <!-- Left wheel joint -->
   <joint name="left_wheel_joint" type="continuous">
     <parent link="base_link"/>
     <child link="left_wheel"/>
-    <origin xyz="-${body_length/3} ${body_width/2 + wheel_width/2} ${wheel_radius/2}" rpy="0 0 0"/>
+    <origin xyz="0 ${body_width/2 + wheel_width/2} 0.05" rpy="0 0 0"/>  <!-- Changed Z from 0 to 0.05 -->
     <axis xyz="0 1 0"/>
   </joint>
+<!-- Right wheel joint -->
   <joint name="right_wheel_joint" type="continuous">
     <parent link="base_link"/>
     <child link="right_wheel"/>
-    <origin xyz="-${body_length/3} -${body_width/2 + wheel_width/2} ${wheel_radius/2}" rpy="0 0 0"/>
+    <origin xyz="0 -${body_width/2 + wheel_width/2} 0.05" rpy="0 0 0"/> <!-- Changed Z from 0 to 0.05 -->
     <axis xyz="0 1 0"/>
   </joint>
   <!-- Front Caster Wheel -->
-  <link name="caster_wheel">
+  <!-- <link name="caster_wheel">
     <visual>
       <geometry>
@@ -125,10 +127,10 @@
       <origin xyz="0 0 0" rpy="0 0 0"/>
     </inertial>
-  </link>
-  <joint name="caster_joint" type="fixed">
+  </link> -->
+  <!-- <joint name="caster_joint" type="fixed">
     <parent link="base_link"/>
     <child link="caster_wheel"/>
     <origin xyz="0.05 0 0" rpy="0 0 0"/>
-  </joint>
+  </joint> -->
   <!-- Camera link -->
   <link name="camera_link">
@@ -146,5 +148,5 @@
     <parent link="base_link"/>
     <child link="camera_link"/>
-    <origin xyz="0.1 0 ${body_height + 0.025}" rpy="0 0 0"/>
+    <origin xyz="${body_length/2 - 0.025} 0 ${1.75*body_height}" rpy="0 0 0"/>
   </joint>
   <!-- Gazebo plugin for camera -->
@@ -176,3 +178,17 @@
     </sensor>
   </gazebo>
+  <gazebo>
+    <plugin name="diff_drive_controller" filename="libgazebo_ros_diff_drive.so">
+      <ros>
+        <remapping>cmd_vel:=/cmd_vel</remapping>
+      </ros>
+      <update_rate>100.0</update_rate>
+      <left_joint>left_wheel_joint</left_joint>
+      <right_joint>right_wheel_joint</right_joint>
+      <wheel_separation>0.2</wheel_separation> <!-- Adjust according to your robot -->
+      <wheel_diameter>0.1</wheel_diameter>
+      <torque>1.0</torque>
+      <command_topic>/cmd_vel</command_topic>
+    </plugin>
+  </gazebo>
 </robot>

Commit message: Added README with setup, launch and build instructions

File: src/vision_line_follower/urdf/my_robot.urdf.xacro (robot description, xacro)
@@ -15,5 +15,5 @@
       </geometry>
       <material name="gray">
-        <color rgba="0.6 0.6 0.6 1.0"/>
+        <color rgba="1.0 0.0 0.0 1.0"/>
       </material>
     </visual>
@@ -32,4 +32,7 @@
     </inertial>
   </link>
+  <gazebo reference="base_link">
+    <material>Gazebo/Red</material>
+  </gazebo>
     <!-- Left wheel -->
     <link name="left_wheel">
